Commit message: amcl e ompl modificati

File: pioneer_p3dx_model/p3dx_description/urdf/pioneer3dx.xacro (robot description, xacro)
@@ -212,5 +212,5 @@
 	<joint name="lms100_joint" type="fixed">
 		<axis xyz="0 1 0" />
-		<origin xyz="0.12 0 0.26" rpy="0 0 0" />
+		<origin xyz="0 0 0.3" rpy="0 0 0" /> <!-- was xyz="0.12 0 0.26" -->
 		<parent link="base_link" />
 		<child link="lms100" />
