Commit message: mannequins now do wander

File: mannequin/urdf/diff_robot.xacro (robot description, xacro)
@@ -3,4 +3,5 @@
   <xacro:include filename="$(find rl_robot_description_pkg)/urdf/diff_robot_macro.xacro" />
   <xacro:property name="M_PI" value="3.1415926535897931" />
+  <xacro:arg name="prefix" default="mann1"/>
 		<!--Actual body/chassis of the robot-->
 	<link name="base_link">
@@ -39,5 +40,5 @@
 			<origin xyz="0 0 0.95" rpy="0 0 0" />
 			<geometry>
-				<cylinder length="1.90" radius="0.5" />
+				<cylinder length="1.90" radius="0.3" />
 			</geometry>
 		</collision>
@@ -48,5 +49,6 @@
 		<origin xyz="0.0 0.0 0.1" rpy="0 0 0"/>
 	</joint>
-	<!--<link name="sensor_link">
+	<link name="sensor_link">
+		<!--
     <collision>
       <origin xyz="0 0 0.05" rpy="0 0 0"/>
@@ -55,11 +57,12 @@
       </geometry>
     </collision>
+		-->
     <visual>
       <origin xyz="0 0 0.05" rpy="0 0 0"/>
       <geometry>
-        <box size="0.1 0.1 0.1"/>
+        <box size="0.01 0.01 0.01"/>
       </geometry>
       <material name="orange"/>
-    </visual>-->
+    </visual>
 		<!--
     <inertial>
@@ -71,11 +74,11 @@
         izz="1.0"/>
     </inertial>
-  </link>
+		-->
+        </link>
 	<joint name="sensor_joint" type="fixed">
-		<parent link="base_link" />
+		<parent link="humanbody" />
 		<child link="sensor_link" />
-		<origin xyz="0.0 0.0 0.1" rpy="0 0 0"/>
+		<origin xyz="0.0 0.0 0.8" rpy="0 0 0"/>
 	</joint>
--->
 	<xacro:caster_joint
 		name="caster_front_link"
@@ -118,7 +121,7 @@
       <wheelTorque>30</wheelTorque>
       <wheelAcceleration>1.8</wheelAcceleration>
-      <commandTopic>cmd_vel</commandTopic>
-      <odometryFrame>odom</odometryFrame>
-      <odometryTopic>odom</odometryTopic>
+      <commandTopic>/$(arg prefix)/cmd_vel</commandTopic>
+      <odometryFrame>/$(arg prefix)/odom</odometryFrame>
+      <odometryTopic>/$(arg prefix)/odom</odometryTopic>
       <robotBaseFrame>base_link</robotBaseFrame>
     </plugin>
@@ -126,3 +129,34 @@
 		</plugin>
   </gazebo>
+  <gazebo reference="sensor_link">
+		<sensor type="ray" name="laser">
+      <pose>0 0 0.0 0 0 0</pose>
+      <visualize>false</visualize>
+      <update_rate>40</update_rate>
+       <ray>
+        <scan>
+          <horizontal>
+            <samples>360</samples>
+            <resolution>1</resolution>
+             <min_angle>-1.57</min_angle>
+             <max_angle>1.57</max_angle>
+          </horizontal>
+        </scan>
+        <range>
+          <min>0.4</min>
+          <max>10.0</max>
+          <resolution>0.0001</resolution>
+        </range>
+        <noise>
+          <type>gaussian</type>
+          <mean>0.0</mean>
+          <stddev>0.0001</stddev>
+        </noise>
+      </ray>
+      <plugin name="gazebo_ros_head_hokuyo_controller" filename="libgazebo_ros_laser.so">
+        <topicName>/$(arg prefix)/laser/scan</topicName>
+        <frameName>base_link</frameName>
+      </plugin>
+		</sensor>
+  </gazebo>
 </robot>

Commit message: files were missing

File: mannequin/urdf/diff_robot.xacro (robot description, xacro)
@@ -1,5 +1,5 @@
 <?xml version="1.0"?>
 <robot name="diff_robot" xmlns:xacro="http://ros.org/wiki/xacro">
-  <xacro:include filename="$(find rl_robot_description_pkg)/urdf/diff_robot_macro.xacro" />
+  <xacro:include filename="$(find mannequin)/urdf/diff_robot_macro.xacro" />
   <xacro:property name="M_PI" value="3.1415926535897931" />
   <xacro:arg name="prefix" default="mann1"/>
@@ -34,5 +34,5 @@
 			<origin xyz="0 0 0" rpy="1.57 0 1.57" />
 			<geometry>
-				<mesh filename="package://rl_robot_description_pkg/meshes/mannequin.dae" />
+				<mesh filename="package://mannequin/meshes/mannequin.dae" />
 			</geometry>
 		</visual>
@@ -79,5 +79,5 @@
 		<parent link="humanbody" />
 		<child link="sensor_link" />
-		<origin xyz="0.0 0.0 0.8" rpy="0 0 0"/>
+		<origin xyz="0.0 0.0 0.3" rpy="0 0 0"/>
 	</joint>
 	<xacro:caster_joint
